Commit message: Feature:
- Add environment variable check to enable Pacejka plugin
Fix:
- steering hinge joint from continuous to revolute
- remove steering dynamics

File: racecar_description/urdf/macros.xacro (robot description, xacro)
@@ -85,17 +85,17 @@
     <cylinder length="0.045" radius="0.05" />
   </geometry>
-  <xacro:unless value="$(optenv PACEJKA true)">
-  <surface>
-    <friction>
-      <ode>
-        <mu>1.0</mu>
-  	<mu2>1.0</mu2>
-        <fdir1>1 0 0</fdir1>
-        <slip1>0</slip1>
-        <slip2>0</slip2>
-      </ode>
-    </friction>
-  </surface>
-  </xacro:unless>
+  <xacro:if value="$(optenv PACEJKA false)">
+   <surface>
+     <friction>
+       <ode>
+         <mu>1.0</mu>
+   	     <mu2>1.0</mu2>
+         <fdir1>1 0 0</fdir1>
+         <slip1>0</slip1>
+         <slip2>0</slip2>
+       </ode>
+     </friction>
+   </surface>
+  </xacro:if>
 </xacro:macro>
 <xacro:macro name="right_wheels_collision_geometry">
@@ -104,17 +104,17 @@
     <cylinder length="0.045" radius="0.05" />
   </geometry>
-  <xacro:unless value="$(optenv PACEJKA true)">
-  <surface>
-    <friction>
-      <ode>
-        <mu>1.0</mu>
-  	<mu2>1.0</mu2>
-        <fdir1>0 0 1</fdir1>
-        <slip1>0</slip1>
-        <slip2>0</slip2>
-      </ode>
-    </friction>
-  </surface>
-  </xacro:unless>
+  <xacro:if value="$(optenv PACEJKA false)">
+   <surface>
+     <friction>
+       <ode>
+         <mu>1.0</mu>
+   	     <mu2>1.0</mu2>
+         <fdir1>0 0 1</fdir1>
+         <slip1>0</slip1>
+         <slip2>0</slip2>
+       </ode>
+     </friction>
+   </surface>
+  </xacro:if>
 </xacro:macro>
 <!-- transmission macros -->

File: racecar_description/urdf/racecar.xacro (robot description, xacro)
@@ -82,5 +82,5 @@
     <child link="left_steering_hinge" />
     <axis xyz="-1 0 0" />
-    <limit lower="-1.0" upper="1.0" effort="10" velocity="100" />
+    <limit lower="-1.0" upper="1.0" effort="1000" velocity="100" />
   </joint>
   <xacro:steering_hinge_transmission name="left_steering_hinge" />
@@ -95,10 +95,10 @@
     </visual>
   </link>
-  <joint name="right_steering_hinge_joint" type="continuous">
+  <joint name="right_steering_hinge_joint" type="revolute">
     <origin xyz="0.325 -0.1 0" rpy="0 1.5708 0" />
     <parent link="chassis" />
     <child link="right_steering_hinge" />
     <axis xyz="-1 0 0" />
-    <limit lower="-1.0" upper="1.0" effort="10" velocity="100" />
+    <limit lower="-1.0" upper="1.0" effort="1000" velocity="100" />
   </joint>
   <xacro:steering_hinge_transmission name="right_steering_hinge" />
